Commit message: feat(rl): complete M2.5 autonomous reinforcement learning pipeline and WebGL integration

File: output/models_archive/gen_01_baseline_confined_v1/evolved_confined_space.urdf (robot description, URDF)
Before this commit: robot evolved_unit_test_inspection, 8 links, 7 joints
Links:
- removed link sensor_0_s_depth_cam
- added link sensor_0_s_lidar_2d, mass 0.1350; visual box size=0.04 0.04 0.04
- added link sensor_1_s_depth_cam, mass 0.0600; visual box size=0.04 0.04 0.04
- link arm_0: geometry visual cylinder length=0.160 radius=0.01
- link arm_1: geometry visual cylinder length=0.160 radius=0.01
- link arm_2: geometry visual cylinder length=0.160 radius=0.01
- link arm_3: geometry visual cylinder length=0.160 radius=0.01
- link arm_4: geometry visual cylinder length=0.160 radius=0.01
- link arm_5: geometry visual cylinder length=0.160 radius=0.01
Joints:
- removed joint joint_base_sensor_0_s_depth_cam
- added joint joint_base_sensor_0_s_lidar_2d: type fixed, parent base_link, child sensor_0_s_lidar_2d, origin xyz=-0.0800 -0.0200 0.0500 rpy=0 0 0
- added joint joint_base_sensor_1_s_depth_cam: type fixed, parent base_link, child sensor_1_s_depth_cam, origin xyz=0.0200 0.0500 0.0500 rpy=0 0 0
- joint joint_base_arm_0: origin xyz=0.1000 0.0000 0.0 rpy=0 1.5708 0.0000 -> xyz=0.0800 0.0000 0.0 rpy=0 1.5708 0.0000
- joint joint_base_arm_1: origin xyz=0.0500 0.0866 0.0 rpy=0 1.5708 1.0472 -> xyz=0.0400 0.0693 0.0 rpy=0 1.5708 1.0472
- joint joint_base_arm_2: origin xyz=-0.0500 0.0866 0.0 rpy=0 1.5708 2.0944 -> xyz=-0.0400 0.0693 0.0 rpy=0 1.5708 2.0944
- joint joint_base_arm_3: origin xyz=-0.1000 0.0000 0.0 rpy=0 1.5708 3.1416 -> xyz=-0.0800 0.0000 0.0 rpy=0 1.5708 3.1416
- joint joint_base_arm_4: origin xyz=-0.0500 -0.0866 0.0 rpy=0 1.5708 4.1888 -> xyz=-0.0400 -0.0693 0.0 rpy=0 1.5708 4.1888
- joint joint_base_arm_5: origin xyz=0.0500 -0.0866 0.0 rpy=0 1.5708 5.2360 -> xyz=0.0400 -0.0693 0.0 rpy=0 1.5708 5.2360

File: output/models_archive/gen_02_agile_confined_v2/evolved_agile_confined_v2.urdf (robot description, URDF)
Before this commit: robot evolved_unit_test_inspection, 8 links, 7 joints
Links:
- removed link arm_4
- removed link arm_5
- removed link sensor_0_s_depth_cam
- added link sensor_0_s_lidar_2d, mass 0.1350; visual box size=0.04 0.04 0.04
- added link sensor_1_s_depth_cam, mass 0.0600; visual box size=0.04 0.04 0.04
- link arm_0: mass 0.0225 -> 0.0640
- link arm_1: mass 0.0225 -> 0.0640
- link arm_2: mass 0.0225 -> 0.0640
- link arm_3: mass 0.0225 -> 0.0640
- link base_link: mass 0.8000 -> 0.2000
Joints:
- removed joint joint_base_arm_4
- removed joint joint_base_arm_5
- removed joint joint_base_sensor_0_s_depth_cam
- added joint joint_base_sensor_0_s_lidar_2d: type fixed, parent base_link, child sensor_0_s_lidar_2d, origin xyz=0.0000 0.0000 0.0600 rpy=0 0 0
- added joint joint_base_sensor_1_s_depth_cam: type fixed, parent base_link, child sensor_1_s_depth_cam, origin xyz=0.1000 0.0000 0.0000 rpy=0 0 0
- joint joint_base_arm_1: origin xyz=0.0500 0.0866 0.0 rpy=0 1.5708 1.0472 -> xyz=0.0000 0.1000 0.0 rpy=0 1.5708 1.5708
- joint joint_base_arm_2: origin xyz=-0.0500 0.0866 0.0 rpy=0 1.5708 2.0944 -> xyz=-0.1000 0.0000 0.0 rpy=0 1.5708 3.1416
- joint joint_base_arm_3: origin xyz=-0.1000 0.0000 0.0 rpy=0 1.5708 3.1416 -> xyz=-0.0000 -0.1000 0.0 rpy=0 1.5708 4.7124
