Commit message: feat(webgl): add BOM drawer, 4 dynamic environments, and crash damage simulation (DIG-8, DIG-9, DIG-10)

File: output/evolved_unit_test_inspection.urdf (robot description, URDF)
Before this commit: robot evolved_unit_test_inspection, 6 links, 5 joints
Links:
- link arm_0: geometry visual cylinder length=0.150 radius=0.01
- link arm_1: geometry visual cylinder length=0.150 radius=0.01
- link arm_2: geometry visual cylinder length=0.150 radius=0.01
- link arm_3: geometry visual cylinder length=0.150 radius=0.01
Joints:
- joint joint_base_arm_0: origin xyz=0.1000 0.0000 0.0 rpy=0 1.5708 0.0000 -> xyz=0.0750 0.0000 0.0 rpy=0 1.5708 0.0000
- joint joint_base_arm_1: origin xyz=0.0000 0.1000 0.0 rpy=0 1.5708 1.5708 -> xyz=0.0000 0.0750 0.0 rpy=0 1.5708 1.5708
- joint joint_base_arm_2: origin xyz=-0.1000 0.0000 0.0 rpy=0 1.5708 3.1416 -> xyz=-0.0750 0.0000 0.0 rpy=0 1.5708 3.1416
- joint joint_base_arm_3: origin xyz=-0.0000 -0.1000 0.0 rpy=0 1.5708 4.7124 -> xyz=-0.0000 -0.0750 0.0 rpy=0 1.5708 4.7124
- joint joint_base_sensor_0_s_depth_cam: origin xyz=0.0900 -0.0900 0.0500 rpy=0 0 0 -> xyz=-0.0400 -0.0400 0.0500 rpy=0 0 0

Commit message: feat(telemetry): add 20Hz flight data recorder and training dataset exporter (DIG-12)

File: output/evolved_unit_test_inspection.urdf (robot description, URDF)
Before this commit: robot evolved_unit_test_inspection, 6 links, 5 joints
Links:
- link arm_0: geometry visual cylinder length=0.160 radius=0.01
- link arm_1: geometry visual cylinder length=0.160 radius=0.01
- link arm_2: geometry visual cylinder length=0.160 radius=0.01
- link arm_3: geometry visual cylinder length=0.160 radius=0.01
Joints:
- joint joint_base_arm_0: origin xyz=0.0750 0.0000 0.0 rpy=0 1.5708 0.0000 -> xyz=0.0800 0.0000 0.0 rpy=0 1.5708 0.0000
- joint joint_base_arm_1: origin xyz=0.0000 0.0750 0.0 rpy=0 1.5708 1.5708 -> xyz=0.0000 0.0800 0.0 rpy=0 1.5708 1.5708
- joint joint_base_arm_2: origin xyz=-0.0750 0.0000 0.0 rpy=0 1.5708 3.1416 -> xyz=-0.0800 0.0000 0.0 rpy=0 1.5708 3.1416
- joint joint_base_arm_3: origin xyz=-0.0000 -0.0750 0.0 rpy=0 1.5708 4.7124 -> xyz=-0.0000 -0.0800 0.0 rpy=0 1.5708 4.7124
- joint joint_base_sensor_0_s_depth_cam: origin xyz=-0.0400 -0.0400 0.0500 rpy=0 0 0 -> xyz=0.1000 -0.0100 0.0500 rpy=0 0 0

Commit message: docs(output): update evolution lineage report and test outputs

File: output/evolved_unit_test_inspection.urdf (robot description, URDF)
Before this commit: robot evolved_unit_test_inspection, 6 links, 5 joints
Links:
- added link arm_4, mass 0.0225; visual cylinder length=0.170 radius=0.01
- added link arm_5, mass 0.0225; visual cylinder length=0.170 radius=0.01
- link arm_0: geometry visual cylinder length=0.170 radius=0.01
- link arm_1: geometry visual cylinder length=0.170 radius=0.01
- link arm_2: geometry visual cylinder length=0.170 radius=0.01
- link arm_3: geometry visual cylinder length=0.170 radius=0.01
Joints:
- added joint joint_base_arm_4: type fixed, parent base_link, child arm_4, origin xyz=-0.0425 -0.0736 0.0 rpy=0 1.5708 4.1888
- added joint joint_base_arm_5: type fixed, parent base_link, child arm_5, origin xyz=0.0425 -0.0736 0.0 rpy=0 1.5708 5.2360
- joint joint_base_arm_0: origin xyz=0.0800 0.0000 0.0 rpy=0 1.5708 0.0000 -> xyz=0.0850 0.0000 0.0 rpy=0 1.5708 0.0000
- joint joint_base_arm_1: origin xyz=0.0000 0.0800 0.0 rpy=0 1.5708 1.5708 -> xyz=0.0425 0.0736 0.0 rpy=0 1.5708 1.0472
- joint joint_base_arm_2: origin xyz=-0.0800 0.0000 0.0 rpy=0 1.5708 3.1416 -> xyz=-0.0425 0.0736 0.0 rpy=0 1.5708 2.0944
- joint joint_base_arm_3: origin xyz=-0.0000 -0.0800 0.0 rpy=0 1.5708 4.7124 -> xyz=-0.0850 0.0000 0.0 rpy=0 1.5708 3.1416
- joint joint_base_sensor_0_s_depth_cam: origin xyz=0.1000 -0.0100 0.0500 rpy=0 0 0 -> xyz=0.0600 -0.0900 0.0500 rpy=0 0 0

Commit message: fix(flight-physics): resolve flight direction anomaly using YXZ aerospace rotation and 3D thrust vectoring (DIG-12)

File: output/evolved_unit_test_inspection.urdf (robot description, URDF)
Before this commit: robot evolved_unit_test_inspection, 8 links, 7 joints
Links:
- link arm_0: geometry visual cylinder length=0.210 radius=0.01
- link arm_1: geometry visual cylinder length=0.210 radius=0.01
- link arm_2: geometry visual cylinder length=0.210 radius=0.01
- link arm_3: geometry visual cylinder length=0.210 radius=0.01
- link arm_4: geometry visual cylinder length=0.210 radius=0.01
- link arm_5: geometry visual cylinder length=0.210 radius=0.01
Joints:
- joint joint_base_arm_0: origin xyz=0.0850 0.0000 0.0 rpy=0 1.5708 0.0000 -> xyz=0.1050 0.0000 0.0 rpy=0 1.5708 0.0000
- joint joint_base_arm_1: origin xyz=0.0425 0.0736 0.0 rpy=0 1.5708 1.0472 -> xyz=0.0525 0.0909 0.0 rpy=0 1.5708 1.0472
- joint joint_base_arm_2: origin xyz=-0.0425 0.0736 0.0 rpy=0 1.5708 2.0944 -> xyz=-0.0525 0.0909 0.0 rpy=0 1.5708 2.0944
- joint joint_base_arm_3: origin xyz=-0.0850 0.0000 0.0 rpy=0 1.5708 3.1416 -> xyz=-0.1050 0.0000 0.0 rpy=0 1.5708 3.1416
- joint joint_base_arm_4: origin xyz=-0.0425 -0.0736 0.0 rpy=0 1.5708 4.1888 -> xyz=-0.0525 -0.0909 0.0 rpy=0 1.5708 4.1888
- joint joint_base_arm_5: origin xyz=0.0425 -0.0736 0.0 rpy=0 1.5708 5.2360 -> xyz=0.0525 -0.0909 0.0 rpy=0 1.5708 5.2360
- joint joint_base_sensor_0_s_depth_cam: origin xyz=0.0600 -0.0900 0.0500 rpy=0 0 0 -> xyz=-0.0400 -0.0400 0.0500 rpy=0 0 0

Commit message: feat(rl): complete M2.5.2 privileged DRL teacher-student distillation with stage inspector

File: output/evolved_unit_test_inspection.urdf (robot description, URDF)
Before this commit: robot evolved_unit_test_inspection, 8 links, 7 joints
Links:
- removed link arm_4
- removed link arm_5
- link arm_0: geometry visual cylinder length=0.210 radius=0.01
- link arm_1: geometry visual cylinder length=0.210 radius=0.01
- link arm_2: geometry visual cylinder length=0.210 radius=0.01
- link arm_3: geometry visual cylinder length=0.210 radius=0.01
Joints:
- removed joint joint_base_arm_4
- removed joint joint_base_arm_5
- joint joint_base_arm_0: origin xyz=0.1000 0.0000 0.0 rpy=0 1.5708 0.0000 -> xyz=0.1050 0.0000 0.0 rpy=0 1.5708 0.0000
- joint joint_base_arm_1: origin xyz=0.0500 0.0866 0.0 rpy=0 1.5708 1.0472 -> xyz=0.0000 0.1050 0.0 rpy=0 1.5708 1.5708
- joint joint_base_arm_2: origin xyz=-0.0500 0.0866 0.0 rpy=0 1.5708 2.0944 -> xyz=-0.1050 0.0000 0.0 rpy=0 1.5708 3.1416
- joint joint_base_arm_3: origin xyz=-0.1000 0.0000 0.0 rpy=0 1.5708 3.1416 -> xyz=-0.0000 -0.1050 0.0 rpy=0 1.5708 4.7124
- joint joint_base_sensor_0_s_depth_cam: origin xyz=-0.0500 -0.0800 0.0500 rpy=0 0 0 -> xyz=0.0500 -0.0900 0.0500 rpy=0 0 0
